File: Hardware/Breakout Board design files/ArduinoRFM95 V6.brd (EAGLE design)
At the start: 53.3 x 35.6 mm, 46 parts, among them J2 AVR_SPI_PRG_6PTH, J3 USB-SMD-NS, Q1 PMV37EN, Q2 MOSFET-NCHANNEL2N7002PW, Q3 PMV48XP, U1 ATMEGA328P_TQFP, U2 RFM69HCW, U3 FT231XS, U4 NCP1117ST50T3G, U5 LP2992-33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

Commit message: update
Parts:
- Q1: value PMV37EN -> FDN360P
- R6, R7: value 10K -> 470R
- moved FRAME1 80.8 mm to (3.81, 43.2)
Changed lines of the file:
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@@
 <attribute name="VALUE" x="31.496" y="31.623" size="0.4064" layer="27" font="vector" rot="R180"/>
 </element>
-<element name="FRAME1" library="SparkFun-Retired" package="CREATIVE_COMMONS" value="FRAME-LETTER" x="-76.2" y="31.75"/>
+<element name="FRAME1" library="SparkFun-Retired" package="CREATIVE_COMMONS" value="FRAME-LETTER" x="3.81" y="43.18"/>
 <element name="J2" library="SparkFun-Connectors" package="2X3" value="AVR_SPI_PRG_6PTH" x="43.18" y="6.35" smashed="yes">
 <attribute name="VALUE" x="41.91" y="3.175" size="1.27" layer="27"/>
@@
 <attribute name="VALUE" x="48.387" y="16.764" size="0.4064" layer="28" font="vector" rot="MR90"/>
 </element>
-<element name="R6" library="SparkFun-Resistors" package="0603-RES" value="10K" x="13.97" y="20.32" smashed="yes">
+<element name="R6" library="SparkFun-Resistors" package="0603-RES" value="470R" x="13.97" y="20.32" smashed="yes">
 <attribute name="VALUE" x="12.954" y="19.177" size="0.4064" layer="27" font="vector"/>
 </element>
-<element name="R7" library="SparkFun-Resistors" package="0603-RES" value="10K" x="13.97" y="22.86" smashed="yes" rot="R180">
+<element name="R7" library="SparkFun-Resistors" package="0603-RES" value="470R" x="13.97" y="22.86" smashed="yes" rot="R180">
 <attribute name="VALUE" x="14.986" y="24.003" size="0.4064" layer="27" font="vector" rot="R180"/>
 </element>
@@
 <attribute name="VALUE" x="18.415" y="24.765" size="1.27" layer="27" rot="R180"/>
 </element>
-<element name="Q1" library="SparkFun-DiscreteSemi" package="SOT23-3" value="PMV37EN" x="19.05" y="6.35" smashed="yes" rot="R270">
+<element name="Q1" library="SparkFun-DiscreteSemi" package="SOT23-3" value="FDN360P" x="19.05" y="6.35" smashed="yes" rot="R270">
 <attribute name="VALUE" x="18.8595" y="7.366" size="0.4064" layer="27" rot="R270"/>
 </element>
